File: TOSLINK Switch for gscartsw.kicad_pcb (KiCad board)
At the start: 2 copper layers, 228.9 x 24 mm, 20 parts, among them U1 8-to-1-MUX, U2 EXT

Commit message: added tantalum cap
Parts:
- added 100μF 7343: CP_Tantalum_Case-D_EIA-7343-31_Hand, Capacitors_Tantalum_SMD:CP_Tantalum_Case-D_EIA-7343-31_Hand, F.Cu at (272.0, 130.3)
Routing:
- net (no net): track 0.00 -> 296.1 mm, vias 0 -> 45
- net GND: track 38.9 -> 2.73 mm, vias 16 -> 0
- net +5V: track 401.9 -> 404.2 mm
